File: Eletronics/Main Board/Main Board.kicad_sch (KiCad schematic)
At the start: 0 parts

Commit message: [ADDED] Main Components
Other:
- removed sheet ESP32 S3 CIRCUIT
- removed sheet Motor Control Circuit
Changed lines of the file:
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@@
-(kicad_sch (version 20211123) (generator eeschema)
+(kicad_sch (version 20230121) (generator eeschema)
   (paper "A4")
   (title_block
@@
     (date "2023-03-19")
   )
-  (sheet (at 184.15 53.34) (size 39.37 25.4) (fields_autoplaced)
-    (stroke (width 0.1524) (type solid) (color 0 0 0 0))
-    (fill (color 215 206 255 1.0000))
-    (property "Sheet name" "Motor Control Circuit" (id 0) (at 184.15 52.6284 0)
+  (sheet (at 154.94 80.01) (size 40.64 24.13) (fields_autoplaced)
+    (stroke (width 0.1524) (type solid))
+    (fill (color 208 247 255 1.0000))
+    (property "Sheetname" "STM32 CIRCUIT" (at 154.94 79.2984 0)
       (effects (font (size 1.27 1.27)) (justify left bottom))
     )
-    (property "Sheet file" "motorcontrolcircuit.kicad_sch" (id 1) (at 184.15 79.3246 0)
+    (property "Sheetfile" "stm32circuit.kicad_sch" (at 154.94 104.7246 0)
       (effects (font (size 1.27 1.27)) (justify left top))
     )
+    (instances
+      (project "Main Board"
+        (path "/9c55052f-48ce-482f-9116-275e8c52377d" (page "3"))
+      )
+    )
   )
-  (sheet (at 59.69 93.98) (size 40.64 24.13)
-    (stroke (width 0.1524) (type solid) (color 0 0 0 0))
-    (fill (color 197 255 205 1.0000))
-    (property "Sheet name" "ESP32 S3 CIRCUIT" (id 0) (at 59.69 93.98 0)
+  (sheet (at 73.66 137.16) (size 40.64 24.13) (fields_autoplaced)
+    (stroke (width 0.1524) (type solid))
+    (fill (color 255 225 137 1.0000))
+    (property "Sheetname" "Peripherals Circuit" (at 73.66 136.4484 0)
       (effects (font (size 1.27 1.27)) (justify left bottom))
     )
-    (property "Sheet file" "ESP32S3.kicad_sch" (id 1) (at 59.69 118.6946 0)
+    (property "Sheetfile" "peripheralscircuit.kicad_sch" (at 73.66 161.8746 0)
       (effects (font (size 1.27 1.27)) (justify left top))
     )
+    (instances
+      (project "Main Board"
+        (path "/9c55052f-48ce-482f-9116-275e8c52377d" (page "5"))
+      )
+    )
   )
-  (sheet (at 185.42 95.25) (size 40.64 24.13) (fields_autoplaced)
-    (stroke (width 0.1524) (type solid) (color 0 0 0 0))
-    (fill (color 208 247 255 1.0000))
-    (property "Sheet name" "STM32 CIRCUIT" (id 0) (at 185.42 94.5384 0)
+  (sheet (at 74.93 24.13) (size 40.64 24.13) (fields_autoplaced)
+    (stroke (width 0.1524) (type solid))
+    (fill (color 255 254 213 1.0000))
+    (property "Sheetname" "Power Circuit" (at 74.93 23.4184 0)
       (effects (font (size 1.27 1.27)) (justify left bottom))
     )
-    (property "Sheet file" "stm32circuit.kicad_sch" (id 1) (at 185.42 119.9646 0)
+    (property "Sheetfile" "powercircuit.kicad_sch" (at 74.93 48.8446 0)
       (effects (font (size 1.27 1.27)) (justify left top))
     )
-  )
-  (sheet (at 123.19 93.98) (size 40.64 24.13) (fields_autoplaced)
-    (stroke (width 0.1524) (type solid) (color 0 0 0 0))
-    (fill (color 255 225 137 1.0000))
-    (property "Sheet name" "Peripherals Circuit" (id 0) (at 123.19 93.2684 0)
-      (effects (font (size 1.27 1.27)) (justify left bottom))
-    )
-    (property "Sheet file" "peripheralscircuit.kicad_sch" (id 1) (at 123.19 118.6946 0)
-      (effects (font (size 1.27 1.27)) (justify left top))
-    )
-  )
-  (sheet (at 120.65 53.34) (size 40.64 24.13) (fields_autoplaced)
-    (stroke (width 0.1524) (type solid) (color 0 0 0 0))
-    (fill (color 255 254 213 1.0000))
-    (property "Sheet name" "Power Circuit" (id 0) (at 120.65 52.6284 0)
-      (effects (font (size 1.27 1.27)) (justify left bottom))
-    )
-    (property "Sheet file" "powercircuit.kicad_sch" (id 1) (at 120.65 78.0546 0)
-      (effects (font (size 1.27 1.27)) (justify left top))
+    (instances
+      (project "Main Board"
+        (path "/9c55052f-48ce-482f-9116-275e8c52377d" (page "4"))
+      )
     )
   )
   (sheet_instances
     (path "/" (page "1"))
-    (path "/8b9a232e-7faa-4988-8c2c-da79f53fb3dd" (page "2"))
-    (path "/d61f1aa0-0047-4ce3-b0b1-dd877d44cec3" (page "3"))
-    (path "/f0117347-2404-40f1-b32d-75bb535cab22" (page "4"))
-    (path "/e376cead-5d62-4603-93fb-b0271804a22a" (page "5"))
-    (path "/7d9e1f2e-3a85-4b38-9cda-6ff66a356245" (page "6"))
-  )
-  (symbol_instances
-    (path "/d61f1aa0-0047-4ce3-b0b1-dd877d44cec3/3ae9eb73-8186-486e-9aaf-1c806c7efbd6"
-      (reference "U?") (unit 1) (value "STM32F103C8Tx") (footprint "Package_QFP:LQFP-48_7x7mm_P0.5mm")
-    )
-    (path "/8b9a232e-7faa-4988-8c2c-da79f53fb3dd/58ccb4f7-e396-4361-880c-0281a46456b1"
-      (reference "U?") (unit 1) (value "ESP32-S3-WROOM-1-N4") (footprint "ESP32WROOM S3:ESP32-S3-WROOM-1-N8")
-    )
   )
 )

Commit message: Perifericos ok
Changed lines of the file:
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@@
     )
   )
-  (sheet (at 73.66 137.16) (size 40.64 24.13) (fields_autoplaced)
+  (sheet (at 78.74 115.57) (size 40.64 24.13) (fields_autoplaced)
     (stroke (width 0.1524) (type solid))
     (fill (color 255 225 137 1.0000))
-    (property "Sheetname" "Peripherals Circuit" (at 73.66 136.4484 0)
+    (property "Sheetname" "Peripherals Circuit" (at 78.74 114.8584 0)
       (effects (font (size 1.27 1.27)) (justify left bottom))
     )
-    (property "Sheetfile" "peripheralscircuit.kicad_sch" (at 73.66 161.8746 0)
+    (property "Sheetfile" "peripheralscircuit.kicad_sch" (at 78.74 140.2846 0)
       (effects (font (size 1.27 1.27)) (justify left top))
     )
@@
     )
   )
-  (sheet (at 74.93 24.13) (size 40.64 24.13) (fields_autoplaced)
+  (sheet (at 76.2 44.45) (size 40.64 24.13) (fields_autoplaced)
     (stroke (width 0.1524) (type solid))
     (fill (color 255 254 213 1.0000))
-    (property "Sheetname" "Power Circuit" (at 74.93 23.4184 0)
+    (property "Sheetname" "Power Circuit" (at 76.2 43.7384 0)
       (effects (font (size 1.27 1.27)) (justify left bottom))
     )
-    (property "Sheetfile" "powercircuit.kicad_sch" (at 74.93 48.8446 0)
+    (property "Sheetfile" "powercircuit.kicad_sch" (at 76.2 69.1646 0)
       (effects (font (size 1.27 1.27)) (justify left top))
     )

Commit message: update sch
Other:
- sheet Peripherals Circuit ports: added CS, INT, LED, SCL, SDA, SDO; removed none
Changed lines of the file:
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@@
       (effects (font (size 1.27 1.27)) (justify left top))
+    )
+    (pin "SDA" input (at 119.38 120.65 0)
+      (effects (font (size 1.27 1.27)) (justify right))
+    )
+    (pin "SDO" input (at 119.38 123.19 0)
+      (effects (font (size 1.27 1.27)) (justify right))
+    )
+    (pin "INT" input (at 119.38 125.73 0)
+      (effects (font (size 1.27 1.27)) (justify right))
+    )
+    (pin "CS" input (at 119.38 129.54 0)
+      (effects (font (size 1.27 1.27)) (justify right))
+    )
+    (pin "SCL" input (at 119.38 132.08 0)
+      (effects (font (size 1.27 1.27)) (justify right))
+    )
+    (pin "LED" input (at 119.38 134.62 0)
+      (effects (font (size 1.27 1.27)) (justify right))
     )
     (instances
