File: Eletronics/Main Board/peripheralscircuit.kicad_sch (KiCad schematic)
At the start: 0 parts

Commit message: [ADDED] Main Components
Parts:
- added D1: WS2812B, LED_SMD:LED_WS2812B_PLCC4_5.0x5.0mm_P3.2mm, symbol LED:WS2812B
- added U4: LSM6DSL, Package_LGA:LGA-14_3x2.5mm_P0.5mm_LayoutBorder3x4y, symbol Sensor_Motion:LSM6DSL
Connections:
- new net: U4.6 (GND), U4.7 (GND)
Changed lines of the file:
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@@
-(kicad_sch (version 20211123) (generator eeschema)
+(kicad_sch (version 20230121) (generator eeschema)
   (paper "A4")
+  (symbol (lib_id "Sensor_Motion:LSM6DSL") (at 151.13 54.61 0) (unit 1)
+    (in_bom yes) (on_board yes) (dnp no) (fields_autoplaced)
+    (property "Reference" "U4" (at 153.0859 69.85 0)
+      (effects (font (size 1.27 1.27)) (justify left))
+    )
+    (property "Value" "LSM6DSL" (at 153.0859 72.39 0)
+      (effects (font (size 1.27 1.27)) (justify left))
+    )
+    (property "Footprint" "Package_LGA:LGA-14_3x2.5mm_P0.5mm_LayoutBorder3x4y" (at 140.97 72.39 0)
+      (effects (font (size 1.27 1.27)) (justify left) hide)
+    )
+    (property "Datasheet" "https://www.st.com/resource/en/datasheet/lsm6dsl.pdf" (at 153.67 71.12 0)
+      (effects (font (size 1.27 1.27)) hide)
+    )
+    (pin "1")
+    (pin "10")
+    (pin "11")
+    (pin "12")
+    (pin "13")
+    (pin "14")
+    (pin "2")
+    (pin "3")
+    (pin "4")
+    (pin "5")
+    (pin "6")
+    (pin "7")
+    (pin "8")
+    (pin "9")
+    (instances
+      (project "Main Board"
+        (path "/9c55052f-48ce-482f-9116-275e8c52377d/e376cead-5d62-4603-93fb-b0271804a22a"
+          (reference "U4") (unit 1)
+        )
+      )
+    )
+  )
+  (symbol (lib_id "LED:WS2812B") (at 55.88 55.88 0) (unit 1)
+    (in_bom yes) (on_board yes) (dnp no) (fields_autoplaced)
+    (property "Reference" "D1" (at 67.31 52.7559 0)
+      (effects (font (size 1.27 1.27)))
+    )
+    (property "Value" "WS2812B" (at 67.31 55.2959 0)
+      (effects (font (size 1.27 1.27)))
+    )
+    (property "Footprint" "LED_SMD:LED_WS2812B_PLCC4_5.0x5.0mm_P3.2mm" (at 57.15 63.5 0)
+      (effects (font (size 1.27 1.27)) (justify left top) hide)
+    )
+    (property "Datasheet" "https://cdn-shop.adafruit.com/datasheets/WS2812B.pdf" (at 58.42 65.405 0)
+      (effects (font (size 1.27 1.27)) (justify left top) hide)
+    )
+    (pin "1")
+    (pin "2")
+    (pin "3")
+    (pin "4")
+    (instances
+      (project "Main Board"
+        (path "/9c55052f-48ce-482f-9116-275e8c52377d/e376cead-5d62-4603-93fb-b0271804a22a"
+          (reference "D1") (unit 1)
+        )
+      )
+    )
+  )
 )

Commit message: Perifericos ok
Parts:
- added C202 (x2): 100nF, symbol Device:C_Small
- added R401, R402: 10k, symbol Device:R_Small
Connections:
- net SDO: now reaches U4.1 (SDO/SA0)
- net CS: now reaches U4.12 (CS)
- net SCL: now reaches U4.13 (SCL)
- net SCL: now also R402.2
- net SDA: now reaches U4.14 (SDA)
- net SDA: now also R401.2
- net GND: now reaches U4.2 (SDX)
- net GND: now also D1.3 (VSS), U4.3 (SCX), U4.6 (GND), U4.7 (GND), C202.2, C202.2
- net INT: now reaches U4.4 (INT1)
- net +3.3V: now reaches U4.5 (VDDIO)
- net +3.3V: now also U4.8 (VDD), C202.1, C202.1, R401.1, R402.1
- net +5V: now reaches D1.1 (VDD)
- net LED: now reaches D1.4 (DIN)
- no-connect marks 0 -> 2
Other:
- note added: "possivel melhoria : colocar 2 acelerometros, 1 bem no centro e outro na borda"
- moved on the sheet: D1, U4

Commit message: update sch
Parts:
- C202: footprint (none) -> Capacitor_SMD:C_0603_1608Metric
- R401, R402: footprint (none) -> Resistor_SMD:R_0603_1608Metric
Changed lines of the file:
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@@
       (effects (font (size 1.27 1.27)) (justify left))
     )
-    (property "Footprint" "" (at 201.93 99.06 0)
+    (property "Footprint" "Resistor_SMD:R_0603_1608Metric" (at 201.93 99.06 0)
       (effects (font (size 1.27 1.27)) hide)
     )
@@
       (effects (font (size 1.27 1.27)) (justify left))
     )
-    (property "Footprint" "" (at 215.9 77.47 0)
+    (property "Footprint" "Capacitor_SMD:C_0603_1608Metric" (at 215.9 77.47 0)
       (effects (font (size 1.27 1.27)) hide)
     )
@@
       (effects (font (size 1.27 1.27)) (justify left))
     )
-    (property "Footprint" "" (at 187.96 99.06 0)
+    (property "Footprint" "Resistor_SMD:R_0603_1608Metric" (at 187.96 99.06 0)
       (effects (font (size 1.27 1.27)) hide)
     )
@@
       (effects (font (size 1.27 1.27)) (justify left))
     )
-    (property "Footprint" "" (at 205.74 77.47 0)
-      (effects (font (size 1.27 1.27)) hide)
-    )
+    (property "Footprint" "Capacitor_SMD:C_0603_1608Metric" (at 205.74 77.47 0)
+      (effects (font (size 1.27 1.27)) hide)
+    )
