File: Eletronics/Main Board/powercircuit.kicad_sch (KiCad schematic)
At the start: 0 parts

Commit message: [ADDED] Main Components
Parts:
- added U1: AMS1117-5.0, Package_TO_SOT_SMD:SOT-223-3_TabPin2, symbol Regulator_Linear:AMS1117-5.0
- added U2: AMS1117-3.3, Package_TO_SOT_SMD:SOT-223-3_TabPin2, symbol Regulator_Linear:AMS1117-3.3
Changed lines of the file:
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@@
-(kicad_sch (version 20211123) (generator eeschema)
+(kicad_sch (version 20230121) (generator eeschema)
   (paper "A4")
+  (symbol (lib_id "Regulator_Linear:AMS1117-3.3") (at 116.84 46.99 0) (unit 1)
+    (in_bom yes) (on_board yes) (dnp no) (fields_autoplaced)
+    (property "Reference" "U2" (at 116.84 40.64 0)
+      (effects (font (size 1.27 1.27)))
+    )
+    (property "Value" "AMS1117-3.3" (at 116.84 43.18 0)
+      (effects (font (size 1.27 1.27)))
+    )
+    (property "Footprint" "Package_TO_SOT_SMD:SOT-223-3_TabPin2" (at 116.84 41.91 0)
+      (effects (font (size 1.27 1.27)) hide)
+    )
+    (property "Datasheet" "http://www.advanced-monolithic.com/pdf/ds1117.pdf" (at 119.38 53.34 0)
+      (effects (font (size 1.27 1.27)) hide)
+    )
+    (pin "1")
+    (pin "2")
+    (pin "3")
+    (instances
+      (project "Main Board"
+        (path "/9c55052f-48ce-482f-9116-275e8c52377d/f0117347-2404-40f1-b32d-75bb535cab22"
+          (reference "U2") (unit 1)
+        )
+      )
+    )
+  )
+  (symbol (lib_id "Regulator_Linear:AMS1117-5.0") (at 82.55 46.99 0) (unit 1)
+    (in_bom yes) (on_board yes) (dnp no) (fields_autoplaced)
+    (property "Reference" "U1" (at 82.55 40.64 0)
+      (effects (font (size 1.27 1.27)))
+    )
+    (property "Value" "AMS1117-5.0" (at 82.55 43.18 0)
+      (effects (font (size 1.27 1.27)))
+    )
+    (property "Footprint" "Package_TO_SOT_SMD:SOT-223-3_TabPin2" (at 82.55 41.91 0)
+      (effects (font (size 1.27 1.27)) hide)
+    )
+    (property "Datasheet" "http://www.advanced-monolithic.com/pdf/ds1117.pdf" (at 85.09 53.34 0)
+      (effects (font (size 1.27 1.27)) hide)
+    )
+    (pin "1")
+    (pin "2")
+    (pin "3")
+    (instances
+      (project "Main Board"
+        (path "/9c55052f-48ce-482f-9116-275e8c52377d/f0117347-2404-40f1-b32d-75bb535cab22"
+          (reference "U1") (unit 1)
+        )
+      )
+    )
+  )
 )

Commit message: Power ok
Parts:
- added C201 (x2): 10uF, symbol Device:C_Small
- added C202 (x2): 22nF, symbol Device:C_Small
Connections:
- net GND: now reaches U2.1 (GND)
- net GND: now also U1.1 (GND), C201.2, C201.2, C202.2, C202.2
- net +3V3: now reaches U2.2 (VO)
- net +3V3: now also C202.1
- net +5V: now reaches U2.3 (VI)
- net +5V: now also U1.2 (VO), C201.1, C202.1
- net +BATT: now reaches U1.3 (VI)
- net +BATT: now also C201.1
Other:
- moved on the sheet: U1, U2

Commit message: update sch
Parts:
- C201, C202: footprint (none) -> Capacitor_SMD:C_0603_1608Metric
Changed lines of the file:
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@@
       (effects (font (size 1.27 1.27)) (justify left))
     )
-    (property "Footprint" "" (at 189.23 100.33 0)
+    (property "Footprint" "Capacitor_SMD:C_0603_1608Metric" (at 189.23 100.33 0)
       (effects (font (size 1.27 1.27)) hide)
     )
@@
       (effects (font (size 1.27 1.27)) (justify left))
     )
-    (property "Footprint" "" (at 134.62 100.33 0)
+    (property "Footprint" "Capacitor_SMD:C_0603_1608Metric" (at 134.62 100.33 0)
       (effects (font (size 1.27 1.27)) hide)
     )
@@
       (effects (font (size 1.27 1.27)) (justify left))
     )
-    (property "Footprint" "" (at 102.87 100.33 0)
+    (property "Footprint" "Capacitor_SMD:C_0603_1608Metric" (at 102.87 100.33 0)
       (effects (font (size 1.27 1.27)) hide)
     )
@@
       (effects (font (size 1.27 1.27)) (justify left))
     )
-    (property "Footprint" "" (at 157.48 100.33 0)
-      (effects (font (size 1.27 1.27)) hide)
-    )
+    (property "Footprint" "Capacitor_SMD:C_0603_1608Metric" (at 157.48 100.33 0)
+      (effects (font (size 1.27 1.27)) hide)
+    )
