File: Eletronics/Main Board/stm32circuit.kicad_sch (KiCad schematic)
At the start: 13 parts, among them U3 STM32F411CEUx, Y201 32.768KHz ±20ppm 6pF, Y202 25MHZ 9PF

Commit message: update sch
Parts:
- removed C206: 10uF, symbol Device:C_Small
- added C1: 2.2uF, Capacitor_SMD:C_0603_1608Metric, symbol Device:C_Small
- C201, C202, C203, C204, C205, C207, C208, C209, C210: footprint (none) -> Capacitor_SMD:C_0603_1608Metric
Connections:
- net GND: now also C1.2
- net at U3.22 (VCAP1): now also C1.1
Changed lines of the file:
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@@
+    (stroke (width 0) (type default))
+  )
+  (wire (pts (xy 92.71 144.78) (xy 92.71 146.05))
     (stroke (width 0) (type default))
   )
@@
     (stroke (width 0) (type default))
   )
+  (wire (pts (xy 92.71 144.78) (xy 104.14 144.78))
+    (stroke (width 0) (type default))
+  )
   (wire (pts (xy 82.55 86.36) (xy 82.55 74.93))
     (stroke (width 0) (type default))
@@
   )
   (wire (pts (xy 44.45 74.93) (xy 53.34 74.93))
+    (stroke (width 0) (type default))
+  )
+  (wire (pts (xy 92.71 151.13) (xy 92.71 152.4))
     (stroke (width 0) (type default))
   )
@@
       (effects (font (size 1.27 1.27)) (justify left))
     )
-    (property "Footprint" "" (at 129.54 34.29 0)
+    (property "Footprint" "Capacitor_SMD:C_0603_1608Metric" (at 129.54 34.29 0)
       (effects (font (size 1.27 1.27)) hide)
     )
@@
       (effects (font (size 1.27 1.27)) (justify left))
     )
-    (property "Footprint" "" (at 138.43 34.29 0)
+    (property "Footprint" "Capacitor_SMD:C_0603_1608Metric" (at 138.43 34.29 0)
       (effects (font (size 1.27 1.27)) hide)
     )
@@
       (effects (font (size 1.27 1.27)) (justify left))
     )
-    (property "Footprint" "" (at 55.88 96.52 0)
+    (property "Footprint" "Capacitor_SMD:C_0603_1608Metric" (at 55.88 96.52 0)
       (effects (font (size 1.27 1.27)) hide)
     )
@@
       (effects (font (size 1.27 1.27)) (justify left))
     )
-    (property "Footprint" "" (at 55.88 74.93 0)
+    (property "Footprint" "Capacitor_SMD:C_0603_1608Metric" (at 55.88 74.93 0)
       (effects (font (size 1.27 1.27)) hide)
     )
@@
         (path "/9c55052f-48ce-482f-9116-275e8c52377d/d61f1aa0-0047-4ce3-b0b1-dd877d44cec3"
           (reference "Y201") (unit 1)
-        )
-      )
-    )
-  )
-  (symbol (lib_id "Device:C_Small") (at 35.56 57.15 0) (unit 1)
-    (in_bom yes) (on_board yes) (dnp no)
-    (property "Reference" "C206" (at 36.83 55.88 0)
-      (effects (font (size 1.27 1.27)) (justify left))
-    )
-    (property "Value" "10uF" (at 36.83 58.42 0)
-      (effects (font (size 1.27 1.27)) (justify left))
-    )
-    (property "Footprint" "" (at 35.56 57.15 0)
-      (effects (font (size 1.27 1.27)) hide)
-    )
-    (property "Datasheet" "~" (at 35.56 57.15 0)
-      (effects (font (size 1.27 1.27)) hide)
-    )
-    (property "LCSC" "" (at 35.56 57.15 0)
-      (effects (font (size 1.27 1.27)) hide)
-    )
-    (pin "1")
-    (pin "2")
-    (instances
-      (project "Main Board"
-        (path "/9c55052f-48ce-482f-9116-275e8c52377d/d61f1aa0-0047-4ce3-b0b1-dd877d44cec3"
-          (reference "C206") (unit 1)
         )
       )
@@
       (effects (font (size 1.27 1.27)) (justify left))
     )
-    (property "Footprint" "" (at 156.21 34.29 0)
+    (property "Footprint" "Capacitor_SMD:C_0603_1608Metric" (at 156.21 34.29 0)
       (effects (font (size 1.27 1.27)) hide)
     )
@@
         (path "/9c55052f-48ce-482f-9116-275e8c52377d/d61f1aa0-0047-4ce3-b0b1-dd877d44cec3"
           (reference "C205") (unit 1)
+        )
+      )
+    )
+  )
+  (symbol (lib_id "Device:C_Small") (at 92.71 148.59 0) (unit 1)
+    (in_bom yes) (on_board yes) (dnp no)
+    (property "Reference" "C1" (at 93.98 147.32 0)
+      (effects (font (size 1.27 1.27)) (justify left))
+    )
+    (property "Value" "2.2uF" (at 93.98 149.86 0)
+      (effects (font (size 1.27 1.27)) (justify left))
+    )
+    (property "Footprint" "Capacitor_SMD:C_0603_1608Metric" (at 92.71 148.59 0)
+      (effects (font (size 1.27 1.27)) hide)
+    )
+    (property "Datasheet" "~" (at 92.71 148.59 0)
+      (effects (font (size 1.27 1.27)) hide)
+    )
+    (property "LCSC" "" (at 92.71 148.59 0)
+      (effects (font (size 1.27 1.27)) hide)
+    )
+    (pin "1")
+    (pin "2")
+    (instances
+      (project "Main Board"
+        (path "/9c55052f-48ce-482f-9116-275e8c52377d/d61f1aa0-0047-4ce3-b0b1-dd877d44cec3"
+          (reference "C1") (unit 1)
         )
       )
@@
       (effects (font (size 1.27 1.27)) (justify left))
     )
-    (property "Footprint" "" (at 55.88 105.41 0)
+    (property "Footprint" "Capacitor_SMD:C_0603_1608Metric" (at 55.88 105.41 0)
       (effects (font (size 1.27 1.27)) hide)
     )
@@
     )
   )
+  (symbol (lib_id "power:GND") (at 92.71 152.4 0) (unit 1)
+    (in_bom yes) (on_board yes) (dnp no) (fields_autoplaced)
+    (property "Reference" "#PWR01" (at 92.71 158.75 0)
+      (effects (font (size 1.27 1.27)) hide)
+    )
+    (property "Value" "GND" (at 92.71 157.48 0)
+      (effects (font (size 1.27 1.27)))
+    )
+    (property "Footprint" "" (at 92.71 152.4 0)
+      (effects (font (size 1.27 1.27)) hide)
+    )
+    (property "Datasheet" "" (at 92.71 152.4 0)
+      (effects (font (size 1.27 1.27)) hide)
+    )
+    (pin "1")
+    (instances
+      (project "Main Board"
+        (path "/9c55052f-48ce-482f-9116-275e8c52377d/d61f1aa0-0047-4ce3-b0b1-dd877d44cec3"
+          (reference "#PWR01") (unit 1)
+        )
+      )
+    )
+  )
   (symbol (lib_id "Device:C_Small") (at 55.88 83.82 90) (unit 1)
     (in_bom yes) (on_board yes) (dnp no)
@@
       (effects (font (size 1.27 1.27)) (justify left))
     )
-    (property "Footprint" "" (at 55.88 83.82 0)
+    (property "Footprint" "Capacitor_SMD:C_0603_1608Metric" (at 55.88 83.82 0)
       (effects (font (size 1.27 1.27)) hide)
     )
@@
       (effects (font (size 1.27 1.27)) (justify left))
     )
-    (property "Footprint" "" (at 120.65 34.29 0)
+    (property "Footprint" "Capacitor_SMD:C_0603_1608Metric" (at 120.65 34.29 0)
       (effects (font (size 1.27 1.27)) hide)
     )
@@
       (effects (font (size 1.27 1.27)) (justify left))
     )
-    (property "Footprint" "" (at 147.32 34.29 0)
-      (effects (font (size 1.27 1.27)) hide)
-    )
+    (property "Footprint" "Capacitor_SMD:C_0603_1608Metric" (at 147.32 34.29 0)
+      (effects (font (size 1.27 1.27)) hide)
+    )
