File: Eletronics/Main Board/stm32circuit.kicad_sch (KiCad schematic)
At the start: 1 part

Commit message: [ADDED] Main Components
Parts:
- removed U?: STM32F103C8Tx, Package_QFP:LQFP-48_7x7mm_P0.5mm, symbol MCU_ST_STM32F1:STM32F103C8Tx
- added U3: STM32F411CEUx, Package_DFN_QFN:QFN-48-1EP_7x7mm_P0.5mm_EP5.6x5.6mm, symbol MCU_ST_STM32F4:STM32F411CEUx
Connections:
- new net: U3.23 (VSS), U3.35 (VSS), U3.47 (VSS), U3.49 (VSS)
Changed lines of the file:
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@@
-(kicad_sch (version 20211123) (generator eeschema)
+(kicad_sch (version 20230121) (generator eeschema)
   (paper "A4")
-  (symbol (lib_id "MCU_ST_STM32F1:STM32F103C8Tx") (at 59.69 99.06 0) (unit 1)
-    (in_bom yes) (on_board yes) (fields_autoplaced)
-    (property "Reference" "U?" (id 0) (at 64.2494 137.16 0)
+  (symbol (lib_id "MCU_ST_STM32F4:STM32F411CEUx") (at 78.74 86.36 0) (unit 1)
+    (in_bom yes) (on_board yes) (dnp no) (fields_autoplaced)
+    (property "Reference" "U3" (at 83.2359 127 0)
       (effects (font (size 1.27 1.27)) (justify left))
     )
-    (property "Value" "STM32F103C8Tx" (id 1) (at 64.2494 139.7 0)
+    (property "Value" "STM32F411CEUx" (at 83.2359 129.54 0)
       (effects (font (size 1.27 1.27)) (justify left))
     )
-    (property "Footprint" "Package_QFP:LQFP-48_7x7mm_P0.5mm" (id 2) (at 44.45 134.62 0)
+    (property "Footprint" "Package_DFN_QFN:QFN-48-1EP_7x7mm_P0.5mm_EP5.6x5.6mm" (at 66.04 124.46 0)
       (effects (font (size 1.27 1.27)) (justify right) hide)
     )
-    (property "Datasheet" "http://www.st.com/st-web-ui/static/active/en/resource/technical/document/datasheet/CD00161566.pdf" (id 3) (at 59.69 99.06 0)
+    (property "Datasheet" "https://www.st.com/resource/en/datasheet/stm32f411ce.pdf" (at 78.74 86.36 0)
       (effects (font (size 1.27 1.27)) hide)
     )
@@
     (pin "47")
     (pin "48")
+    (pin "49")
     (pin "5")
     (pin "6")
@@
     (pin "8")
     (pin "9")
+    (instances
+      (project "Main Board"
+        (path "/9c55052f-48ce-482f-9116-275e8c52377d/d61f1aa0-0047-4ce3-b0b1-dd877d44cec3"
+          (reference "U3") (unit 1)
+        )
+      )
+    )
   )
 )

Commit message: Perifericos ok
Parts:
- added C201: 10uF, symbol Device:C_Small
- added C202, C203, C204, C205: 100nF, symbol Device:C_Small
Connections:
- new net +3V3: C201.1, C202.1, C203.1, C204.1, C205.1
- new net GND: C201.2, C202.2, C203.2, C204.2, C205.2
Changed lines of the file:
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@@
 (kicad_sch (version 20230121) (generator eeschema)
   (paper "A4")
+  (junction (at 129.54 31.75) (diameter 0) (color 0 0 0 0)
+  )
+  (junction (at 120.65 31.75) (diameter 0) (color 0 0 0 0)
+  )
+  (junction (at 147.32 36.83) (diameter 0) (color 0 0 0 0)
+  )
+  (junction (at 129.54 36.83) (diameter 0) (color 0 0 0 0)
+  )
+  (junction (at 147.32 31.75) (diameter 0) (color 0 0 0 0)
+  )
+  (junction (at 138.43 36.83) (diameter 0) (color 0 0 0 0)
+  )
+  (junction (at 138.43 31.75) (diameter 0) (color 0 0 0 0)
+  )
+  (junction (at 120.65 36.83) (diameter 0) (color 0 0 0 0)
+  )
+  (wire (pts (xy 120.65 31.75) (xy 129.54 31.75))
+    (stroke (width 0) (type default))
+  )
+  (wire (pts (xy 129.54 31.75) (xy 138.43 31.75))
+    (stroke (width 0) (type default))
+  )
+  (wire (pts (xy 120.65 36.83) (xy 129.54 36.83))
+    (stroke (width 0) (type default))
+  )
+  (wire (pts (xy 138.43 31.75) (xy 147.32 31.75))
+    (stroke (width 0) (type default))
+  )
+  (wire (pts (xy 147.32 31.75) (xy 156.21 31.75))
+    (stroke (width 0) (type default))
+  )
+  (wire (pts (xy 138.43 36.83) (xy 147.32 36.83))
+    (stroke (width 0) (type default))
+  )
+  (wire (pts (xy 120.65 36.83) (xy 120.65 39.37))
+    (stroke (width 0) (type default))
+  )
+  (wire (pts (xy 147.32 36.83) (xy 156.21 36.83))
+    (stroke (width 0) (type default))
+  )
+  (wire (pts (xy 129.54 36.83) (xy 138.43 36.83))
+    (stroke (width 0) (type default))
+  )
+  (wire (pts (xy 120.65 29.21) (xy 120.65 31.75))
+    (stroke (width 0) (type default))
+  )
+  (symbol (lib_id "Device:C_Small") (at 129.54 34.29 0) (unit 1)
+    (in_bom yes) (on_board yes) (dnp no)
+    (property "Reference" "C202" (at 130.81 33.02 0)
+      (effects (font (size 1.27 1.27)) (justify left))
+    )
+    (property "Value" "100nF" (at 130.81 35.56 0)
+      (effects (font (size 1.27 1.27)) (justify left))
+    )
+    (property "Footprint" "" (at 129.54 34.29 0)
+      (effects (font (size 1.27 1.27)) hide)
+    )
+    (property "Datasheet" "~" (at 129.54 34.29 0)
+      (effects (font (size 1.27 1.27)) hide)
+    )
+    (property "LCSC" "" (at 129.54 34.29 0)
+      (effects (font (size 1.27 1.27)) hide)
+    )
+    (pin "1")
+    (pin "2")
+    (instances
+      (project "Main Board"
+        (path "/9c55052f-48ce-482f-9116-275e8c52377d/d61f1aa0-0047-4ce3-b0b1-dd877d44cec3"
+          (reference "C202") (unit 1)
+        )
+      )
+    )
+  )
+  (symbol (lib_id "Device:C_Small") (at 138.43 34.29 0) (unit 1)
+    (in_bom yes) (on_board yes) (dnp no)
+    (property "Reference" "C203" (at 139.7 33.02 0)
+      (effects (font (size 1.27 1.27)) (justify left))
+    )
+    (property "Value" "100nF" (at 139.7 35.56 0)
+      (effects (font (size 1.27 1.27)) (justify left))
+    )
+    (property "Footprint" "" (at 138.43 34.29 0)
+      (effects (font (size 1.27 1.27)) hide)
+    )
+    (property "Datasheet" "~" (at 138.43 34.29 0)
+      (effects (font (size 1.27 1.27)) hide)
+    )
+    (property "LCSC" "" (at 138.43 34.29 0)
+      (effects (font (size 1.27 1.27)) hide)
+    )
+    (pin "1")
+    (pin "2")
+    (instances
+      (project "Main Board"
+        (path "/9c55052f-48ce-482f-9116-275e8c52377d/d61f1aa0-0047-4ce3-b0b1-dd877d44cec3"
+          (reference "C203") (unit 1)
+        )
+      )
+    )
+  )
+  (symbol (lib_id "power:+3V3") (at 120.65 29.21 0) (unit 1)
+    (in_bom yes) (on_board yes) (dnp no) (fields_autoplaced)
+    (property "Reference" "#PWR0202" (at 120.65 33.02 0)
+      (effects (font (size 1.27 1.27)) hide)
+    )
+    (property "Value" "+3V3" (at 120.65 25.4 0)
+      (effects (font (size 1.27 1.27)))
+    )
+    (property "Footprint" "" (at 120.65 29.21 0)
+      (effects (font (size 1.27 1.27)) hide)
+    )
+    (property "Datasheet" "" (at 120.65 29.21 0)
+      (effects (font (size 1.27 1.27)) hide)
+    )
+    (pin "1")
+    (instances
+      (project "Main Board"
+        (path "/9c55052f-48ce-482f-9116-275e8c52377d/d61f1aa0-0047-4ce3-b0b1-dd877d44cec3"
+          (reference "#PWR0202") (unit 1)
+        )
+      )
+    )
+  )
   (symbol (lib_id "MCU_ST_STM32F4:STM32F411CEUx") (at 78.74 86.36 0) (unit 1)
     (in_bom yes) (on_board yes) (dnp no) (fields_autoplaced)
@@
         )
       )
+    )
+  )
+  (symbol (lib_id "Device:C_Small") (at 156.21 34.29 0) (unit 1)
+    (in_bom yes) (on_board yes) (dnp no)
+    (property "Reference" "C205" (at 157.48 33.02 0)
+      (effects (font (size 1.27 1.27)) (justify left))
+    )
+    (property "Value" "100nF" (at 157.48 35.56 0)
+      (effects (font (size 1.27 1.27)) (justify left))
+    )
+    (property "Footprint" "" (at 156.21 34.29 0)
+      (effects (font (size 1.27 1.27)) hide)
+    )
+    (property "Datasheet" "~" (at 156.21 34.29 0)
+      (effects (font (size 1.27 1.27)) hide)
+    )
+    (property "LCSC" "" (at 156.21 34.29 0)
+      (effects (font (size 1.27 1.27)) hide)
+    )
+    (pin "1")
+    (pin "2")
+    (instances
+      (project "Main Board"
+        (path "/9c55052f-48ce-482f-9116-275e8c52377d/d61f1aa0-0047-4ce3-b0b1-dd877d44cec3"
+          (reference "C205") (unit 1)
+        )
+      )
+    )
+  )
+  (symbol (lib_id "power:GND") (at 120.65 39.37 0) (unit 1)
+    (in_bom yes) (on_board yes) (dnp no) (fields_autoplaced)
+    (property "Reference" "#PWR0201" (at 120.65 45.72 0)
+      (effects (font (size 1.27 1.27)) hide)
+    )
+    (property "Value" "GND" (at 120.65 44.45 0)
+      (effects (font (size 1.27 1.27)))
+    )
+    (property "Footprint" "" (at 120.65 39.37 0)
+      (effects (font (size 1.27 1.27)) hide)
+    )
+    (property "Datasheet" "" (at 120.65 39.37 0)
+      (effects (font (size 1.27 1.27)) hide)
+    )
+    (pin "1")
+    (instances
+      (project "Main Board"
+        (path "/9c55052f-48ce-482f-9116-275e8c52377d/d61f1aa0-0047-4ce3-b0b1-dd877d44cec3"
+          (reference "#PWR0201") (unit 1)
+        )
+      )
+    )
+  )
+  (symbol (lib_id "Device:C_Small") (at 120.65 34.29 0) (unit 1)
+    (in_bom yes) (on_board yes) (dnp no)
+    (property "Reference" "C201" (at 121.92 33.02 0)
+      (effects (font (size 1.27 1.27)) (justify left))
+    )
+    (property "Value" "10uF" (at 121.92 35.56 0)
+      (effects (font (size 1.27 1.27)) (justify left))
+    )
+    (property "Footprint" "" (at 120.65 34.29 0)
+      (effects (font (size 1.27 1.27)) hide)
+    )
+    (property "Datasheet" "~" (at 120.65 34.29 0)
+      (effects (font (size 1.27 1.27)) hide)
+    )
+    (property "LCSC" "" (at 120.65 34.29 0)
+      (effects (font (size 1.27 1.27)) hide)
+    )
+    (pin "1")
+    (pin "2")
+    (instances
+      (project "Main Board"
+        (path "/9c55052f-48ce-482f-9116-275e8c52377d/d61f1aa0-0047-4ce3-b0b1-dd877d44cec3"
+          (reference "C201") (unit 1)
+        )
+      )
+    )
+  )
+  (symbol (lib_id "Device:C_Small") (at 147.32 34.29 0) (unit 1)
+    (in_bom yes) (on_board yes) (dnp no)
+    (property "Reference" "C204" (at 148.59 33.02 0)
+      (effects (font (size 1.27 1.27)) (justify left))
+    )
+    (property "Value" "100nF" (at 148.59 35.56 0)
+      (effects (font (size 1.27 1.27)) (justify left))
+    )
+    (property "Footprint" "" (at 147.32 34.29 0)
+      (effects (font (size 1.27 1.27)) hide)
+    )
+    (property "Datasheet" "~" (at 147.32 34.29 0)
+      (effects (font (size 1.27 1.27)) hide)
+    )
+    (property "LCSC" "" (at 147.32 34.29 0)
+      (effects (font (size 1.27 1.27)) hide)
+    )
+    (pin "1")
+    (pin "2")
+    (instances
+      (project "Main Board"
+        (path "/9c55052f-48ce-482f-9116-275e8c52377d/d61f1aa0-0047-4ce3-b0b1-dd877d44cec3"
+          (reference "C204") (unit 1)
+        )
+      )

Commit message: Power ok
Parts:
- added C206: 10uF, symbol Device:C_Small
- added C207, C208: 4.3pF, symbol Device:C_Small
- added C209, C210: 12 pF, symbol Device:C_Small
- added Y201: 32.768KHz ±20ppm 6pF, symbol Device:Crystal
- added Y202: 25MHZ 9PF, symbol Device:Crystal
Connections:
- net GND: now also C207.1, C208.1, C209.1, C210.1
- net at U3.3 (PC14): now also C207.2, Y201.1
- net at U3.4 (PC15): now also C208.2, Y201.2
- net at U3.5 (PH0): now also C209.2, Y202.1
- net at U3.6 (PH1): now also C210.2, Y202.2
Other:
- moved on the sheet: U3

Commit message: Power ok
Parts:
- added C211: 2.2uF, symbol Device:C_Small
- added C212: 100nF, symbol Device:C_Small
- added FB201: FerriteBead_Small, symbol Device:FerriteBead_Small
- added R201: R_US, symbol Device:R_US
- added R202: 10k, symbol Device:R_US
- added R203: NC, symbol Device:R_US
- added SW201, SW202, SW203: SW_SPST, symbol Switch:SW_SPST
- C206: value 10uF -> 100uF
Connections:
- net +3V3: now also C212.1, R203.1, SW201.2 (B)
- net GND: now also C206.2, C211.2, C212.2, R201.2, R202.2, SW202.2 (B), SW203.2 (B)
- net NRST: now reaches C206.1
- net NRST: now also U3.7 (NRST), R203.2, SW202.1 (A)
- net at U3.1 (VBAT): now also U3.24 (VDD), U3.36 (VDD), U3.48 (VDD), FB201.1
- net PA0: now reaches U3.10 (PA0)
- net PA0: now also SW203.1 (A)
- net at U3.20 (PB2): now also R202.1
- net at U3.22 (VCAP1): now also C211.1
- net BOOT0: now reaches U3.44 (BOOT0)
- net BOOT0: now also R201.1, SW201.1 (A)
- net at U3.9 (VDDA): now also FB201.2
