File: Eletronics/Comunication Board/Comunication Board.kicad_pcb (KiCad board)
At the start: 2 copper layers, 39.5 x 40.1 mm, 36 parts, among them J1 USB_C_Receptacle_USB2.0, J2 Conn_01x10_Female, T1 AMS1117/3V3, U1 BATERIA, U2 ESP32-S3-WROOM-1-N8R2

Commit message: alteracoes finais
Connections:
- U2 pad 41_10: (no net) -> GNDREF
- U2 pad 41_11: (no net) -> GNDREF
- U2 pad 41_12: (no net) -> GNDREF
- U2 pad 41_13: (no net) -> GNDREF
- U2 pad 41_14: (no net) -> GNDREF
- U2 pad 41_15: (no net) -> GNDREF
- U2 pad 41_16: (no net) -> GNDREF
- U2 pad 41_17: (no net) -> GNDREF
- U2 pad 41_18: (no net) -> GNDREF
- U2 pad 41_19: (no net) -> GNDREF
- U2 pad 41_20: (no net) -> GNDREF
- U2 pad 41_21: (no net) -> GNDREF
Routing:
- net +3.3V: track 56.7 -> 47.9 mm, vias 5 -> 8
- net Net-(C1-Pad1): track 20.8 -> 25.0 mm
- net I00: track 58.0 -> 56.2 mm, vias 2 -> 4
- net USB_D+: track 13.1 -> 11.8 mm
- net USB_D-: track 16.5 -> 15.2 mm
- net GNDREF: vias 15 -> 16
- added copper zone on F.Cu, net +3.3V

Commit message: Comunication Board Errors solved
Parts:
- renumbered H4 to H1, H4 to H2, H4 to H3
Routing:
- net GNDREF: track 4.84 -> 27.4 mm, vias 16 -> 17
- net +3.3V: track 47.9 -> 51.3 mm
