File: Eletronics/Comunication Board/Comunication Board.kicad_pcb (KiCad board)
At the start: 2 copper layers, 39.5 x 38.9 mm, 32 parts, among them J1 USB_C_Receptacle_USB2.0, J2 Conn_01x16_Socket, T1 AMS1117/3V3, U1 VCC, U2 ESP32-S3-WROOM-1-N8R2

Commit message: revisão e pequenos ajustes de roteamento
Routing:
- net SPI_CS: track 22.4 -> 25.2 mm
- net GPIO9: track 21.2 -> 23.8 mm
- net SPI_MOSI: track 18.0 -> 20.3 mm
- net USB_D+: track 13.8 -> 16.1 mm
- net SPI_CLK: track 19.8 -> 21.6 mm
- net SPI_MISO: track 15.5 -> 16.8 mm
- net RXD0: track 9.41 -> 10.4 mm
- net GPIO14: track 17.4 -> 18.3 mm
- net GPIO21: track 13.2 -> 13.7 mm
- net GNDREF: vias 4 -> 16
- removed copper zone on B.Cu, net +3.3V
- removed copper zone on F.Cu, net +3.3V

Commit message: fix for manufacture
Parts:
- removed BOOT1: SW_Push, Button_Switch_SMD:SW_SPST_TL3305A
- added EN1: SW_Push, Button_Switch_SMD:SW_SPST_TL3305A, F.Cu at (132.7, 82.9)
- D2: footprint Diode_SMD:D_SMA -> Diode_SMD:D_SOD-123F
- J1: footprint Connector_USB:USB_C_Receptacle_HRO_TYPE-C-31-M-12 -> usb_type_C:USB_C_Receptacle_KH-TYPE-C-16P
- moved J1 0.93 mm to (131.0, 90.8)
- moved D2 0.18 mm to (140.9, 93.7)
- moved R3 0.17 mm to (138.1, 93.2)
Routing:
- net GNDREF: track 16.5 -> 18.8 mm
- net Net-(D2-A): track 22.2 -> 23.7 mm, vias 2 -> 3
- net USB_D-: track 16.1 -> 14.7 mm
- net Net-(J1-CC2): track 2.12 -> 3.05 mm
Other:
- board text added: "SSL Comms V1"
- board text removed: "SSL V1"

Commit message: small fixes
Routing:
- net SPI_CS: track 25.2 -> 27.0 mm
- net SPI_MOSI: track 20.3 -> 21.5 mm
- net GPIO14: track 18.3 -> 17.3 mm
- net SPI_CLK: track 21.6 -> 22.5 mm
- net GPIO9: track 23.8 -> 24.4 mm
- net GPIO21: track 13.7 -> 13.2 mm
- net GNDREF: vias 16 -> 20
