File: Eletronics/Comunication Board/Comunication Board.kicad_sch (KiCad schematic)
At the start: 0 parts

Commit message: Revisão com alterações apontadas no esquemático
Other:
- company: (none) -> Project Neon
- title: (none) -> Placa de comunicação
Changed lines of the file:
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@@
 	(generator_version "8.0")
 	(paper "A4")
+	(title_block
+		(title "Placa de comunicação")
+		(date "2024-05-04")
+		(rev "0")
+		(company "Project Neon")
+		(comment 1 "Autor: Leticia Martins")
+		(comment 2 "Revisão: Marcus Holanda")
+		(comment 3 "Documento com alterações necessárias, não é um docuemnto final")
+	)
 	(sheet
 		(at 206.629 114.3)
