File: Eletronics/Comunication Board/ESP32_S3.kicad_sch (KiCad schematic)
At the start: 1 part, among them U2 ESP32-S3-WROOM-1-N8R2

Commit message: Revisão com alterações apontadas no esquemático
Other:
- company: (none) -> Project Neon
- title: (none) -> Placa de comunicação
Changed lines of the file:
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@@
 	(generator_version "8.0")
 	(paper "A4")
+	(title_block
+		(title "Placa de comunicação")
+		(date "2024-05-04")
+		(rev "0")
+		(company "Project Neon")
+		(comment 1 "Autor: Leticia Martins")
+		(comment 2 "Revisão: Marcus Holanda")
+		(comment 3 "Documento com alterações necessárias, não é um docuemnto final")
+	)
 	(no_connect
 		(at 135.509 110.236)
@@
 		(at 165.989 102.616)
 	)
+	(text_box "Deixar os seguintes pinos disponiveis na barra de pinos:\nIO48,\nIO47,\nIO21,\nIO14,\nIO9"
+		(exclude_from_sim no)
+		(at 213.36 59.69 0)
+		(size 26.67 44.45)
+		(stroke
+			(width 0)
+			(type default)
+		)
+		(fill
+			(type none)
+		)
+		(effects
+			(font
+				(size 1.27 1.27)
+			)
+			(justify left top)
+		)
+	)
 	(global_label "SCL"
