File: Eletronics/Comunication Board/ESP32_S3.kicad_sch (KiCad schematic)
At the start: 1 part, among them U2 ESP32-S3-WROOM-1-N8R2

Commit message: Atualização do repositório
Connections:
- net GPIO14: now reaches U2.22 (IO14)
- net GPIO21: now reaches U2.23 (IO21)
- net GPIO47: now reaches U2.24 (IO47)
- net GPIO48: now reaches U2.25 (IO48)
- no-connect marks 23 -> 19
Other:
- company: Project Neon -> (none)
- title: Placa de comunicação -> (none)
Changed lines of the file:
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@@
 	(generator_version "8.0")
 	(paper "A4")
-	(title_block
-		(title "Placa de comunicação")
-		(date "2024-05-04")
-		(rev "0")
-		(company "Project Neon")
-		(comment 1 "Autor: Leticia Martins")
-		(comment 2 "Revisão: Marcus Holanda")
-		(comment 3 "Documento com alterações necessárias, não é um docuemnto final")
-	)
-	(no_connect
-		(at 135.509 110.236)
-	)
 	(no_connect
 		(at 135.509 82.296)
@@
 	)
 	(no_connect
-		(at 165.989 84.836)
-	)
-	(no_connect
 		(at 135.509 89.916)
 	)
@@
 	)
 	(no_connect
-		(at 165.989 115.316)
-	)
-	(no_connect
 		(at 165.989 77.216)
 	)
@@
 	)
 	(no_connect
-		(at 165.989 112.776)
-	)
-	(no_connect
 		(at 165.989 94.996)
 	)
@@
 		(at 165.989 102.616)
 	)
-	(text_box "Deixar os seguintes pinos disponiveis na barra de pinos:\nIO48,\nIO47,\nIO21,\nIO14,\nIO9"
-		(exclude_from_sim no)
-		(at 213.36 59.69 0)
-		(size 26.67 44.45)
-		(stroke
-			(width 0)
-			(type default)
-		)
-		(fill
-			(type none)
-		)
-		(effects
-			(font
-				(size 1.27 1.27)
-			)
-			(justify left top)
-		)
-	)
 	(global_label "SCL"
 		(shape input)
@@
 		)
 	)
+	(global_label "GPIO48"
+		(shape input)
+		(at 165.989 115.316 0)
+		(fields_autoplaced yes)
+		(effects
+			(font
+				(size 1.27 1.27)
+			)
+			(justify left)
+		)
+		(property "Intersheetrefs" "${INTERSHEET_REFS}"
+			(at 175.8685 115.316 0)
+			(effects
+				(font
+					(size 1.27 1.27)
+				)
+				(justify left)
+				(hide yes)
+			)
+		)
+	)
 	(global_label "TXD0"
 		(shape input)
@@
 		)
 	)
+	(global_label "GPIO47"
+		(shape input)
+		(at 165.989 112.776 0)
+		(fields_autoplaced yes)
+		(effects
+			(font
+				(size 1.27 1.27)
+			)
+			(justify left)
+		)
+		(property "Intersheetrefs" "${INTERSHEET_REFS}"
+			(at 175.8685 112.776 0)
+			(effects
+				(font
+					(size 1.27 1.27)
+				)
+				(justify left)
+				(hide yes)
+			)
+		)
+	)
 	(global_label "RXD0"
 		(shape input)
@@
 		)
 	)
+	(global_label "GPIO14"
+		(shape input)
+		(at 135.509 110.236 180)
+		(fields_autoplaced yes)
+		(effects
+			(font
+				(size 1.27 1.27)
+			)
+			(justify right)
+		)
+		(property "Intersheetrefs" "${INTERSHEET_REFS}"
+			(at 125.6295 110.236 0)
+			(effects
+				(font
+					(size 1.27 1.27)
+				)
+				(justify right)
+				(hide yes)
+			)
+		)
+	)
 	(global_label "SDA"
 		(shape input)
@@
 		)
 		(property "Intersheetrefs" "${INTERSHEET_REFS}"
-			(at 127.4111 97.4566 0)
-			(effects
-				(font
-					(size 1.27 1.27)
-				)
-				(justify right)
-				(hide yes)
-			)
+			(at 126.839 97.536 0)
+			(effects
+				(font
+					(size 1.27 1.27)
+				)
+				(justify right)
+				(hide yes)
+			)
+		)
+	)
+	(global_label "GPIO21"
+		(shape input)
+		(at 165.989 84.836 0)
+		(fields_autoplaced yes)
+		(effects
+			(font
+				(size 1.27 1.27)
+			)
+			(justify left)
+		)
+		(property "Intersheetrefs" "${INTERSHEET_REFS}"
+			(at 175.8685 84.836 0)
+			(effects
+				(font
+					(size 1.27 1.27)
+				)
+				(justify left)
+				(hide yes)
+			)
