File: Eletronics/Comunication Board/USB.kicad_sch (KiCad schematic)
At the start: 6 parts, among them J1 USB_C_Receptacle_USB2.0

Commit message: small fixes
Parts:
- D2: footprint Diode_SMD:D_SMA -> Diode_SMD:D_SOD-123F
- J1: footprint Connector_USB:USB_C_Receptacle_HRO_TYPE-C-31-M-12 -> usb_type_C:USB_C_Receptacle_KH-TYPE-C-16P
Changed lines of the file:
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@@
 			)
 		)
-		(property "Footprint" "Diode_SMD:D_SMA"
+		(property "Footprint" "Diode_SMD:D_SOD-123F"
 			(at 175.26 64.135 0)
 			(effects
@@
 		)
 		(instances
-			(project ""
+			(project "Comunication Board"
 				(path "/4c7888e1-33c4-4d9e-9379-8d84ea02e710/5e8a06e2-a335-4ba3-808d-a5ad2b04f309"
 					(reference "D2")
@@
 			)
 		)
-		(property "Footprint" "Connector_USB:USB_C_Receptacle_HRO_TYPE-C-31-M-12"
+		(property "Footprint" "usb_type_C:USB_C_Receptacle_KH-TYPE-C-16P"
 			(at 129.413 83.82 0)
 			(effects
