File: Eletronics/Comunication Board/Power.kicad_sch (KiCad schematic)
At the start: 8 parts, among them T1 AMS1117/3V3, U1 BATERIA

Commit message: Atualização do repositório
Parts:
- removed POWER1: ON/OFF, Button_Switch_THT:SW_DIP_SPSTx01_Slide_6.7x4.1mm_W7.62mm_P2.54mm_LowProfile, symbol Switch:SW_Push
- removed R4: 1.5 KΩ, Resistor_SMD:R_0603_1608Metric, symbol Device:R_Small
- C6: Field5 (none) -> verificar valor
- C7: value 10 uF -> 22 uF
- L4: Field5 (none) -> Verificar -- outras formas -- Olhar valor do diodo se utili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
- R7: value 330 Ω -> 130 Ω
- T1: Field5 (none) -> precisa?
- U1: value BATERIA -> VCC
Connections:
- net +3.3V: now also R7.1
- net +5V: now also U1.1; no longer R7.1
Other:
- note removed: "Mover Led para lado 3.3V"
- company: Project Neon -> (none)
- title: Placa de comunicação -> (none)
- moved on the sheet: C6, C7, L4, R7, T1, U1
