File: Eletronics/Comunication Board/External.kicad_sch (KiCad schematic)
At the start: 7 parts, among them J2 Conn_01x10_Female

Commit message: Atualização do repositório
Parts:
- removed BZ1: Buzzer, Buzzer_Beeper:Buzzer_12x9.5RM7.6, symbol Device:Buzzer
- removed J2: Conn_01x10_Female, Connector_IDC:IDC-Header_2x05_P2.54mm_Vertical, symbol Connector:Conn_01x10_Female
- removed R11: 330 Ω, Resistor_SMD:R_0603_1608Metric, symbol Device:R_Small
- added J2: Conn_01x16_Socket, Connector_IDC:IDC-Header_2x08_P2.54mm_Vertical, symbol Connector:Conn_01x16_Socket
Connections:
- net GNDREF: now also J2.14 (Pin_14)
- net GPIO9: now also J2.13 (Pin_13)
- net RXD0: now also J2.3 (Pin_3)
- net SCL: now also J2.1 (Pin_1)
- net SDA: now also J2.2 (Pin_2)
- net SPI_CLK: now also J2.10 (Pin_10)
- net SPI_CS: now also J2.12 (Pin_12)
- net SPI_MISO: now also J2.9 (Pin_9)
- net SPI_MOSI: now also J2.11 (Pin_11)
- net TXD0: now also J2.4 (Pin_4)
- new net +5V: J2.15 (Pin_15)
- new net GPIO14: J2.8 (Pin_8)
- new net GPIO21: J2.7 (Pin_7)
- new net GPIO47: J2.6 (Pin_6)
- new net GPIO48: J2.5 (Pin_5)
- no-connect marks 0 -> 1
Other:
- company: Project Neon -> (none)
- title: Placa de comunicação -> (none)
- moved on the sheet: L1, R1, R8, R9
