File: Eletronics/Kicker/Kicker.kicad_pcb (KiCad board)
At the start: 2 copper layers, 37.9 x 20.5 mm, 12 parts, among them J1 Solenoid, J2 Signal, J3 Battery, Q1 IRF540N

Commit message: Kicker modified
Parts:
- added F2: Fuse_Polarized, Fuse:Fuse_Bourns_MF-RG300, F.Cu at (131.7, 63.2)
- moved J2 13.8 mm to (152.6, 61.0), turned to 180 degrees
- moved R1 13.0 mm to (149.8, 63.3)
- moved J1 9.82 mm to (142.7, 69.3)
- moved Q1 5.44 mm to (146.2, 63.4), turned to 180 degrees
- moved D1 3.51 mm to (134.2, 67.5)
- moved G 3.33 mm to (141.2, 56.8)
- moved J3 1.40 mm to (124.2, 65.9), turned to 0 degrees
- moved H4 0.50 mm to (152.2, 68.7)
- moved H4 0.48 mm to (119.2, 68.7)
- moved C1 0.14 mm to (123.1, 56.5)
- moved H4 0.12 mm to (119.2, 53.6)
Connections:
- C1 pad 1: +BATT -> Net-(D1-K)
- D1 pad 1: +BATT -> Net-(D1-K)
- J1 pad 1: +BATT -> Net-(D1-K)
Routing:
- net Net-(D1-K): track 0.00 -> 34.4 mm
- net +BATT: track 28.6 -> 8.61 mm
- net Net-(D1-A): track 31.9 -> 24.5 mm
- net Net-(J2-Pin_1): track 8.37 -> 7.39 mm
Other:
- board size 37.9 x 20.5 mm -> 37.8 x 20 mm

Commit message: kicker modification
Parts:
- moved J1 2.49 mm to (140.2, 69.3)
Routing:
- net Net-(D1-A): track 24.5 -> 29.9 mm
- net Net-(D1-K): track 34.4 -> 32.7 mm
Changed lines of the file:
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@@
+			)
+		)
+		(property "Field5" "+"
+			(at 0 0 180)
+			(unlocked yes)
+			(layer "F.Fab")
+			(hide yes)
+			(effects
+				(font
+					(size 1 1)
+					(thickness 0.15)
+				)
+			)
+		)
+		(property "Field6" "-"
+			(at 0 0 180)
+			(unlocked yes)
+			(layer "F.Fab")
+			(hide yes)
+			(effects
+				(font
+					(size 1 1)
+					(thickness 0.15)
+				)
 			)
 		)
@@
 	(footprint "Connector_PinSocket_2.54mm:PinSocket_1x02_P2.54mm_Vertical"
 		(layer "F.Cu")
-		(at 142.66 69.265 90)
+		(at 140.17 69.275 90)
 		(descr "Through hole straight socket strip, 1x02, 2.54mm pitch, single row (from Kicad 4.0.7), script generated")
 		(tags "Through hole socket strip THT 1x02 2.54mm single row")
@@
 				(font
 					(size 1.27 1.27)
+				)
+			)
+		)
+		(property "+" "+"
+			(at 0 0 90)
+			(unlocked yes)
+			(layer "F.Fab")
+			(hide yes)
+			(effects
+				(font
+					(size 1 1)
+					(thickness 0.15)
+				)
+			)
+		)
+		(property "-" "-"
+			(at 0 0 90)
+			(unlocked yes)
+			(layer "F.Fab")
+			(hide yes)
+			(effects
+				(font
+					(size 1 1)
+					(thickness 0.15)
 				)
 			)
@@
 				(font
 					(size 1.27 1.27)
+				)
+			)
+		)
+		(property "Field5" "+"
+			(at 0 0 0)
+			(unlocked yes)
+			(layer "F.Fab")
+			(hide yes)
+			(effects
+				(font
+					(size 1 1)
+					(thickness 0.15)
+				)
+			)
+		)
+		(property "Field6" "-"
+			(at 0 0 0)
+			(unlocked yes)
+			(layer "F.Fab")
+			(hide yes)
+			(effects
+				(font
+					(size 1 1)
+					(thickness 0.15)
 				)
 			)
@@
 	)
 	(segment
-		(start 145.2 69.265)
-		(end 145.2 68.705)
-		(width 1)
-		(layer "F.Cu")
-		(net 1)
-	)
-	(segment
-		(start 145.2 68.705)
-		(end 143.61 67.115)
-		(width 1)
-		(layer "F.Cu")
-		(net 1)
-	)
-	(segment
 		(start 148.07 56.47)
 		(end 148.01 56.47)
@@
 	)
 	(segment
-		(start 148.01 56.47)
-		(end 143.68 60.8)
+		(start 143.68 63.38)
+		(end 143.68 68.305)
 		(width 1)
 		(layer "F.Cu")
@@
 	)
 	(segment
-		(start 143.524488 63.38)
-		(end 139.384488 67.52)
+		(start 136.1925 67.52)
+		(end 141.515 67.52)
 		(width 1)
 		(layer "F.Cu")
@@
 	)
 	(segment
-		(start 143.61 67.115)
-		(end 143.61 63.45)
+		(start 143.68 68.305)
+		(end 142.71 69.275)
 		(width 1)
 		(layer "F.Cu")
@@
 	)
 	(segment
-		(start 143.68 60.8)
-		(end 143.68 63.38)
-		(width 1)
-		(layer "F.Cu")
-		(net 1)
-	)
-	(segment
-		(start 139.384488 67.52)
-		(end 136.1925 67.52)
+		(start 142.71 68.715)
+		(end 142.71 69.275)
 		(width 1)
 		(layer "F.Cu")
@@
 	)
 	(segment
+		(start 141.515 67.52)
+		(end 142.71 68.715)
+		(width 1)
+		(layer "F.Cu")
+		(net 1)
+	)
+	(segment
+		(start 148.07 65.117081)
+		(end 143.912081 69.275)
+		(width 1)
+		(layer "B.Cu")
+		(net 1)
+	)
+	(segment
+		(start 143.912081 69.275)
+		(end 142.71 69.275)
+		(width 1)
+		(layer "B.Cu")
+		(net 1)
+	)
+	(segment
+		(start 148.07 56.47)
+		(end 148.07 65.117081)
+		(width 1)
+		(layer "B.Cu")
+		(net 1)
+	)
+	(segment
 		(start 147.135 62.465)
 		(end 146.22 63.38)
@@
 	)
 	(segment
-		(start 133.08 67.52)
-		(end 132.1925 67.52)
+		(start 129.19 56.47)
+		(end 136.8 64.08)
 		(width 1)
 		(layer "F.Cu")
@@
 	)
 	(segment
-		(start 134.0825 69.41)
-		(end 142.515 69.41)
-		(width 1)
-		(layer "F.Cu")
-		(net 5)
-	)
-	(segment
-		(start 132.1925 67.52)
-		(end 134.0825 69.41)
-		(width 1)
-		(layer "F.Cu")
-		(net 5)
-	)
-	(segment
-		(start 129.19 56.47)
-		(end 136.8 64.08)
+		(start 133.9475 69.275)
+		(end 132.1925 67.52)
 		(width 1)
 		(layer "F.Cu")
@@
 	)
 	(segment
-		(start 142.515 69.41)
-		(end 142.66 69.265)
+		(start 140.17 69.275)
+		(end 133.9475 69.275)
 		(width 1)
 		(layer "F.Cu")
@@
 	)
 	(segment
-		(start 136.24 64.36)
-		(end 133.08 67.52)
+		(start 140.17 69.275)
+		(end 140.17 67.73)
 		(width 1)
-		(layer "F.Cu")
+		(layer "B.Cu")
+		(net 5)
+	)
+	(segment
+		(start 140.17 67.73)
+		(end 136.8 64.36)
+		(width 1)
+		(layer "B.Cu")
 		(net 5)
 	)
@@
 		(polygon
 			(pts
-				(xy 153.75 71.16) (xy 117.63 71.29) (xy 116.65 69.87) (xy 116.58 52.37) (xy 118.19 50.89) (xy 152.33 50.89)
-				(xy 153.62 51.32) (xy 154.86 52.74) (xy 154.98 55.2) (xy 154.86 69.56) (xy 153.71 71.14) (xy 153.71 71.16)
-				(xy 153.5 71.17) (xy 153.5 71.16)
-			)
-		)
+				(xy 153.685 50.52) (xy 154.925 51.835) (xy 155.12 68.98) (xy 154.145 70.935) (xy 152.19 71.68) (xy 127.87 71.68)
+				(xy 118.385 71.855) (xy 115.68 70.13) (xy 115.91 64.9) (xy 115.855 58.575) (xy 116.255 52.365) (xy 118.155 50.125)
+				(xy 153.665 50.505)
+			)
+		)
