File: Eletronics/Kicker/Kicker.kicad_sch (KiCad schematic)
At the start: 7 parts, among them J1 Solenoid, J2 Signal, J3 Battery, Q1 IRF540N

Commit message: Kicker modified
Parts:
- added F2: Fuse_Polarized, Fuse:Fuse_Bourns_MF-RG300, symbol Device:Fuse_Polarized
Connections:
- net +BATT: now also F2.1; no longer C1.1, D1.1 (K), J1.1 (Pin_1)
- new net: C1.1, D1.1 (K), F2.2, J1.1 (Pin_1)

Commit message: kicker modification
Parts:
- added D2: 1N4007, Diode_SMD:D_SMA, symbol Diode:1N4007
- F2: Field5 (none) -> *Definir ampare** -- 1,5A
- J1: + (none) -> +; - (none) -> -
- J2, J3: Field5 (none) -> +; Field6 (none) -> -
- R1: value 1K -> 130 Ω
Connections:
- net +BATT: now also D2.2 (A); no longer F2.1
- net GNDREF: now also C1.2; no longer R1.2
- net at Q1.1 (G), R1.1: no longer J2.1 (Pin_1)
- net at D1.2 (A), J1.2 (Pin_2), Q1.2 (D): no longer C1.2
- new net: D2.1 (K), F2.1
- new net: J2.1 (Pin_1), R1.2
Other:
- moved on the sheet: C1, J1, R1
